File: Arduino-Pro-v16.sch (EAGLE design)
At the start: 10 parts, among them Q1 RESONATORSMD, U1 ATMEGA328

Commit message: Added the _real_ files for the board
Parts:
- added C2: 0.1uF, SparkFun-Capacitors:CAP0603-CAP
- added C4: (no value), SparkFun-Capacitors:CAP_POL3528
- added J1: (no value), SparkFun-Connectors:M02PTH
- added LED2: Green, LilyPad-Wearables:LED1206
- added R1: 1K, SparkFun-Passives:RESISTOR0603-RES
- added R2: 10K, SparkFun-Passives:RESISTOR0603-RES
- added U$1: TACTILE-SWITCH-7914G, GeekAmmo:TACTILE-SWITCH-7914G
Connections:
- net AREF renamed N$6
- new net DTR: C2.1
- new net N$1: LED2.A, R1.1
- net GND: now also C4.-, J1.1, U$1.1, U$1.2
- net MISO: now also U1.PB4(MISO)
- net MOSI: now also U1.PB3(MOSI/OC2)
- net RESET: now also C2.2, R2.1, U$1.3, U$1.4, U1.PC6(/RESET)
- net SCK: now also R1.2, U1.PB5(SCK)
- net VCC: now also C4.+, J1.2, R2.2
Other:
- note added: "Input Voltage and Ground Connection"
- moved on the sheet: C1, C10, C13, C3, LED1, R11

Commit message: working on schematic
Parts:
- removed C4: (no value), SparkFun-Capacitors:CAP_POL3528
- removed J1: (no value), SparkFun-Connectors:M02PTH
- removed Q1: RESONATORSMD, SparkFun:RESONATORSMD
- removed U$1: TACTILE-SWITCH-7914G, GeekAmmo:TACTILE-SWITCH-7914G
- removed U1: ATMEGA328, SparkFun:ATMEGA168
- added C5: 0.1uF, SparkFun:CAP0402-CAP
- added C6: 0.1uF, SparkFun-Capacitors:CAP0603-CAP
- added D1: (no value), DiscreteComponents:DIODE-DO-214AC
- added FRAME1: FRAME-LETTER, SparkFun-Aesthetics:FRAME-LETTER
- added I2C_PIN, SPI_PIN: (no value), SparkFun-Connectors:M05PTH
- added IC1: ATMEGA1281-16AU, atmel-2005:ATMEGA1281-16AU
- added LED3: Yellow, SparkFun:LED0603
- added LED4: Blue, SparkFun:LED0603
- added LED5: Red, SparkFun:LED0603
- added PWM1, PWM2, PWM3: (no value), SparkFun-Connectors:M04PTH
- added R13, R14, R15, R16, R8, R9: 10K, SparkFun:RESISTOR0402-RES
- added R3: 10K, SparkFun-Passives:RESISTOR0603-RES
- added R4, R5: 220, SparkFun:RESISTOR0402-RES
- added SERIAL1, SERIAL2: (no value), SparkFun-Connectors:M03PTH
- added T1: (no value), DiscreteComponents:FDN340P
- added U$2: TACTILE-SWITCH-7914G, GeekAmmo:TACTILE-SWITCH-7914G
- added U$3, U$4, U$6: BSS138, DiscreteComponents:BSS138
- added Y1: (no value), SparkFun-FreqCtrl:CRYSTALHC49US
- C1: value 0.1uF -> (none); device SparkFun:CAP0402-CAP -> SparkFun-Capacitors:CAP0603-CAP
- C2: value 0.1uF -> (none)
- LED2: device LilyPad-Wearables:LED1206 -> SparkFun:LED0603
- R1: value 1K -> 220; device SparkFun-Passives:RESISTOR0603-RES -> SparkFun:RESISTOR0402-RES
- R2: value 10K -> 220; device SparkFun-Passives:RESISTOR0603-RES -> SparkFun:RESISTOR0402-RES
Connections:
- new net 3V3: R13.2, R15.2, R8.2, U$3.G, U$4.G, U$6.G
- new net 3V3CLK: PCB1.GPIO11, R15.1, U$6.S
- new net 3V3MISO: PCB1.GPIO9, R8.1, U$3.S
- new net 3V3MOSI: PCB1.GPIO10, R13.1, U$4.S
- new net 5VCLK: R16.1, U$6.D
- new net 5VMISO: IC1.(MISO/PCINT3)PB3, R9.1, U$3.D
- new net 5VMOSI: IC1.(MOSI/PCINT2)PB2, R14.1, U$4.D
- new net 5VPROGRAMMER: JP3.2, T1.D
- new net 5VROV: D1.A, T1.G
- new net 5VSCK: IC1.(SCK/PCINT1)PB1
- new net N$10: IC1.(A14)PC6, LED3.A
- new net N$11: IC1.(A15)PC7, LED2.A
- new net N$12: PWM1.3
- new net N$13: PWM1.4
- new net N$14: LED5.C, R1.2
- new net N$15: LED4.C, R2.2
- new net N$16: LED3.C, R4.2
- new net N$17: PWM2.4
- new net N$18: PWM3.1
- new net N$19: PWM3.2
- new net N$2: SERIAL1.1
- new net N$20: PWM3.3
- new net N$21: PWM3.4
- new net N$22: LED2.C, R5.2
- new net N$5: IC1.(A12)PC4, LED5.A
- new net N$7: C5.2, IC1.AREF
- new net N$8: SERIAL2.2
- new net N$9: IC1.(A13)PC5, LED4.A
- new net PWM0A: IC1.(OC0A/OC1C/PCINT7)PB7, PWM1.1
- new net PWM0B: IC1.(OC0B)PG5, PWM1.2
- new net PWM1A: IC1.(OC1A/PCINT5)PB5, PWM2.1
- new net PWM1B: IC1.(OC1B/PCINT6)PB6, PWM2.2
- new net PWM1C: PWM2.3
- new net PWM2A: IC1.(OC2A/PCINT4)PB4
- new net PWM3A: IC1.(OC3A/AIN1)PE3
- new net PWM3B: IC1.(OC3B/INT4)PE4
- new net PWM3C: IC1.(OC3C/INT5)PE5
- new net SCL: I2C_PIN.3, IC1.(SCL/INT0)PD0
- new net SDA: I2C_PIN.2, IC1.(SDA/INT1)PD1
- new net VCCA: PCB1.3V3@1
- net DTR: now also C6.1; no longer C2.1
- net GND: now also C1.2, C2.2, C5.1, I2C_PIN.4, I2C_PIN.5, IC1.AGND, IC1.GND, IC1.GND1, R1.1, R2.1, R4.1, R5.1, SERIAL1.3, SERIAL2.3, SPI_PIN.5, U$2.1, U$2.2; no longer C1.1, C4.-, J1.1, Q1.2, U$1.1, U$1.2, U1.AGND, U1.GND@1, U1.GND@2
- net MISO: now also SPI_PIN.2; no longer U1.PB4(MISO)
- net MOSI: now also SPI_PIN.3; no longer U1.PB3(MOSI/OC2)
- net N$1: now also C1.1, IC1.XTAL1, Y1.2; no longer LED2.A, R1.1
- net N$3: now also C2.1, IC1.XTAL2, Y1.1; no longer Q1.1, U1.PB7(XTAL2/TOSC2)
- net N$4: now also SERIAL1.2; no longer Q1.3, U1.PB6(XTAL1/TOSC1)
- net N$6: now also SERIAL2.1; no longer C1.2, U1.AREF
- net RESET: now also C6.2, IC1.RESET, R3.1, U$2.3, U$2.4; no longer C2.2, R2.1, U$1.3, U$1.4, U1.PC6(/RESET)
- net SCK: now also SPI_PIN.4; no longer R1.2, U1.PB5(SCK)
- net VCC: now also D1.C, I2C_PIN.1, IC1.AVCC, IC1.VCC, IC1.VCC1, R14.2, R16.2, R3.2, R9.2, SPI_PIN.1, T1.S; no longer C4.+, J1.2, JP3.2, R2.2, U1.AVCC, U1.VCC@1, U1.VCC@2
Other:
- note removed: "Input Voltage and Ground Connection"
- moved on the sheet: C1, C2, JP3, LED2, R1, R2

Commit message: Modified power inputs and added a todo list
Parts:
- removed C6: 0.1uF, SparkFun-Capacitors:CAP0603-CAP
Connections:
- removed net DTR: C6.1
- net GND: now also PCB1.GND@14, PCB1.GND@20, PCB1.GND@25, PCB1.GND@30, PCB1.GND@34, PCB1.GND@39, PCB1.GND@6, PCB1.GND@9
- net RESET: no longer C6.2
- net VCCA: now also PCB1.5V@2, PCB1.5V@4; no longer PCB1.3V3@1
Changed lines of the file:
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@@
 <?xml version="1.0" encoding="utf-8"?>
 <!DOCTYPE eagle SYSTEM "eagle.dtd">
-<eagle version="7.6.0">
+<eagle version="7.3.0">
 <drawing>
 <settings>
@@
 <part name="P+4" library="SparkFun" deviceset="VCC" device=""/>
 <part name="R3" library="SparkFun-Passives" deviceset="RESISTOR" device="0603-RES" value="10K"/>
-<part name="C6" library="SparkFun-Capacitors" deviceset="CAP" device="0603-CAP" value="0.1uF"/>
 <part name="U$2" library="GeekAmmo" deviceset="TACTILE-SWITCH" device="-7914G"/>
 <part name="GND12" library="SparkFun" deviceset="GND" device=""/>
@@
 <part name="VCC2" library="SparkFun-Aesthetics" deviceset="VCCA" device=""/>
 <part name="3V2" library="SparkFun-Aesthetics" deviceset="VCCA" device=""/>
-<part name="3V4" library="SparkFun-Aesthetics" deviceset="VCCA" device=""/>
 <part name="U$4" library="DiscreteComponents" deviceset="BSS138" device=""/>
 <part name="R13" library="SparkFun" deviceset="RESISTOR" device="0402-RES" value="10K"/>
@@
 <part name="VCC4" library="SparkFun-Aesthetics" deviceset="VCCA" device=""/>
 <part name="3V3" library="SparkFun-Aesthetics" deviceset="VCCA" device=""/>
+<part name="GND15" library="SparkFun" deviceset="GND" device=""/>
+<part name="GND16" library="SparkFun" deviceset="GND" device=""/>
+<part name="GND17" library="SparkFun" deviceset="GND" device=""/>
+<part name="GND18" library="SparkFun" deviceset="GND" device=""/>
+<part name="GND19" library="SparkFun" deviceset="GND" device=""/>
+<part name="5VROV1" library="SparkFun-Aesthetics" deviceset="VCCA" device=""/>
 </parts>
 <sheets>
@@
 <instance part="P+4" gate="1" x="-218.44" y="177.8"/>
 <instance part="R3" gate="G$1" x="-218.44" y="170.18" rot="R90"/>
-<instance part="C6" gate="G$1" x="-226.06" y="160.02" rot="R90"/>
 <instance part="U$2" gate="G$1" x="-218.44" y="147.32" rot="R90"/>
 <instance part="GND12" gate="1" x="-215.9" y="137.16" rot="MR0"/>
@@
 <instance part="VCC2" gate="G$1" x="76.2" y="106.68" smashed="yes"/>
 <instance part="3V2" gate="G$1" x="50.8" y="106.68" smashed="yes"/>
-<instance part="3V4" gate="G$1" x="304.8" y="127" smashed="yes"/>
 <instance part="U$4" gate="G$1" x="66.04" y="55.88"/>
 <instance part="R13" gate="G$1" x="50.8" y="60.96" rot="R90"/>
@@
 <instance part="VCC4" gate="G$1" x="76.2" y="38.1" smashed="yes"/>
 <instance part="3V3" gate="G$1" x="50.8" y="38.1" smashed="yes"/>
+<instance part="GND15" gate="1" x="406.4" y="121.92"/>
+<instance part="GND16" gate="1" x="370.84" y="121.92"/>
+<instance part="GND17" gate="1" x="386.08" y="162.56"/>
+<instance part="GND18" gate="1" x="347.98" y="162.56"/>
+<instance part="GND19" gate="1" x="330.2" y="121.92"/>
+<instance part="5VROV1" gate="G$1" x="312.42" y="162.56" smashed="yes"/>
 </instances>
 <busses>
@@
 <wire x1="-91.44" y1="86.36" x2="-91.44" y2="83.82" width="0.1524" layer="91"/>
 </segment>
+<segment>
+<pinref part="PCB1" gate="G$1" pin="GND@14"/>
+<wire x1="340.36" y1="154.94" x2="340.36" y2="165.1" width="0.1524" layer="91"/>
+<pinref part="GND18" gate="1" pin="GND"/>
+<wire x1="340.36" y1="165.1" x2="347.98" y2="165.1" width="0.1524" layer="91"/>
+<pinref part="PCB1" gate="G$1" pin="GND@20"/>
+<wire x1="347.98" y1="165.1" x2="355.6" y2="165.1" width="0.1524" layer="91"/>
+<wire x1="355.6" y1="165.1" x2="355.6" y2="154.94" width="0.1524" layer="91"/>
+<junction x="347.98" y="165.1"/>
+<pinref part="PCB1" gate="G$1" pin="GND@6"/>
+<wire x1="320.04" y1="154.94" x2="320.04" y2="165.1" width="0.1524" layer="91"/>
+<wire x1="320.04" y1="165.1" x2="340.36" y2="165.1" width="0.1524" layer="91"/>
+<junction x="340.36" y="165.1"/>
+</segment>
+<segment>
+<pinref part="PCB1" gate="G$1" pin="GND@30"/>
+<wire x1="381" y1="154.94" x2="381" y2="165.1" width="0.1524" layer="91"/>
+<pinref part="GND17" gate="1" pin="GND"/>
+<wire x1="381" y1="165.1" x2="386.08" y2="165.1" width="0.1524" layer="91"/>
+<pinref part="PCB1" gate="G$1" pin="GND@34"/>
+<wire x1="386.08" y1="165.1" x2="391.16" y2="165.1" width="0.1524" layer="91"/>
+<wire x1="391.16" y1="165.1" x2="391.16" y2="154.94" width="0.1524" layer="91"/>
+<junction x="386.08" y="165.1"/>
+</segment>
+<segment>
+<pinref part="PCB1" gate="G$1" pin="GND@25"/>
+<pinref part="GND16" gate="1" pin="GND"/>
+<wire x1="370.84" y1="127" x2="370.84" y2="124.46" width="0.1524" layer="91"/>
+</segment>
+<segment>
+<pinref part="PCB1" gate="G$1" pin="GND@39"/>
+<pinref part="GND15" gate="1" pin="GND"/>
+<wire x1="406.4" y1="127" x2="406.4" y2="124.46" width="0.1524" layer="91"/>
+</segment>
+<segment>
+<pinref part="PCB1" gate="G$1" pin="GND@9"/>
+<pinref part="GND19" gate="1" pin="GND"/>
+<wire x1="330.2" y1="127" x2="330.2" y2="124.46" width="0.1524" layer="91"/>
+</segment>
 </net>
 <net name="RESET" class="0">
@@
 </segment>
 <segment>
-<pinref part="C6" gate="G$1" pin="2"/>
 <wire x1="-187.96" y1="160.02" x2="-215.9" y2="160.02" width="0.1524" layer="91"/>
 <pinref part="U$2" gate="G$1" pin="3"/>
 <wire x1="-215.9" y1="160.02" x2="-218.44" y2="160.02" width="0.1524" layer="91"/>
-<wire x1="-218.44" y1="160.02" x2="-223.52" y2="160.02" width="0.1524" layer="91"/>
 <wire x1="-218.44" y1="152.4" x2="-218.44" y2="160.02" width="0.1524" layer="91"/>
 <junction x="-218.44" y="160.02"/>
@@
 </segment>
 </net>
-<net name="DTR" class="0">
-<segment>
-<pinref part="C6" gate="G$1" pin="1"/>
-<wire x1="-231.14" y1="160.02" x2="-233.68" y2="160.02" width="0.1524" layer="91"/>
-<label x="-233.68" y="160.02" size="1.778" layer="95"/>
-</segment>
-</net>
 <net name="N$7" class="0">
 <segment>
@@
 </segment>
 </net>
-<net name="VCCA" class="0">
-<segment>
-<pinref part="3V4" gate="G$1" pin="VCCA"/>
-<wire x1="304.8" y1="127" x2="304.8" y2="124.46" width="0.1524" layer="91"/>
-<wire x1="304.8" y1="124.46" x2="309.88" y2="124.46" width="0.1524" layer="91"/>
-<pinref part="PCB1" gate="G$1" pin="3V3@1"/>
-<wire x1="309.88" y1="124.46" x2="309.88" y2="127" width="0.1524" layer="91"/>
-</segment>
-</net>
 <net name="5VMOSI" class="0">
 <segment>
@@
 </segment>
 </net>
+<net name="VCCA" class="0">
+<segment>
+<pinref part="PCB1" gate="G$1" pin="5V@2"/>
+<wire x1="309.88" y1="154.94" x2="309.88" y2="162.56" width="0.1524" layer="91"/>
+<pinref part="5VROV1" gate="G$1" pin="VCCA"/>
+<wire x1="309.88" y1="162.56" x2="312.42" y2="162.56" width="0.1524" layer="91"/>
+<pinref part="PCB1" gate="G$1" pin="5V@4"/>
+<wire x1="312.42" y1="162.56" x2="314.96" y2="162.56" width="0.1524" layer="91"/>
+<wire x1="314.96" y1="162.56" x2="314.96" y2="154.94" width="0.1524" layer="91"/>
+<junction x="312.42" y="162.56"/>
+</segment>
+</net>

Commit message: Added JTAG pins and smaller pushbutton
Parts:
- removed U$2: TACTILE-SWITCH-7914G, GeekAmmo:TACTILE-SWITCH-7914G
- added JTAG_CONNECTOR: MICRO-FIT-4-SMD-PART, Connectors:MICRO-FIT-4-SMD-PART
- added U$1: SWITCH, DiscreteComponents:SWITCH
Connections:
- new net JTTCK: IC1.(ADC4/TCK)PF4, JTAG_CONNECTOR.C4
- new net JTTDI: IC1.(ADC7/TDI)PF7, JTAG_CONNECTOR.C1
- new net JTTDO: IC1.(ADC6/TDO)PF6, JTAG_CONNECTOR.C2
- new net JTTMS: IC1.(ADC5/TMS)PF5, JTAG_CONNECTOR.C3
- net GND: now also U$1.P$1; no longer U$2.1, U$2.2
- net RESET: now also U$1.P$2; no longer U$2.3, U$2.4
Changed lines of the file:
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@@
 <?xml version="1.0" encoding="utf-8"?>
 <!DOCTYPE eagle SYSTEM "eagle.dtd">
-<eagle version="7.3.0">
+<eagle version="7.6.0">
 <drawing>
 <settings>
@@
 <part name="P+4" library="SparkFun" deviceset="VCC" device=""/>
 <part name="R3" library="SparkFun-Passives" deviceset="RESISTOR" device="0603-RES" value="10K"/>
-<part name="U$2" library="GeekAmmo" deviceset="TACTILE-SWITCH" device="-7914G"/>
 <part name="GND12" library="SparkFun" deviceset="GND" device=""/>
 <part name="Y1" library="SparkFun-FreqCtrl" deviceset="CRYSTAL" device="HC49US"/>
@@
 <part name="GND19" library="SparkFun" deviceset="GND" device=""/>
 <part name="5VROV1" library="SparkFun-Aesthetics" deviceset="VCCA" device=""/>
+<part name="U$1" library="DiscreteComponents" deviceset="SWITCH" device=""/>
+<part name="JTAG_CONNECTOR" library="Connectors" deviceset="MICRO-FIT-4-SMD" device="" technology="-PART"/>
 </parts>
 <sheets>
@@
 <instance part="P+4" gate="1" x="-218.44" y="177.8"/>
 <instance part="R3" gate="G$1" x="-218.44" y="170.18" rot="R90"/>
-<instance part="U$2" gate="G$1" x="-218.44" y="147.32" rot="R90"/>
-<instance part="GND12" gate="1" x="-215.9" y="137.16" rot="MR0"/>
+<instance part="GND12" gate="1" x="-218.44" y="137.16" rot="MR0"/>
 <instance part="Y1" gate="G$1" x="-193.04" y="152.4" rot="R270"/>
 <instance part="C1" gate="G$1" x="-198.12" y="147.32" rot="R270"/>
@@
 <instance part="GND19" gate="1" x="330.2" y="121.92"/>
 <instance part="5VROV1" gate="G$1" x="312.42" y="162.56" smashed="yes"/>
+<instance part="U$1" gate="G$1" x="-218.44" y="149.86" rot="R90"/>
+<instance part="JTAG_CONNECTOR" gate="G$1" x="-104.14" y="43.18" rot="R270"/>
 </instances>
 <busses>
@@
 <pinref part="C5" gate="G$1" pin="1"/>
 <pinref part="GND8" gate="1" pin="GND"/>
-</segment>
-<segment>
-<pinref part="U$2" gate="G$1" pin="1"/>
-<wire x1="-218.44" y1="142.24" x2="-218.44" y2="139.7" width="0.1524" layer="91"/>
-<pinref part="GND12" gate="1" pin="GND"/>
-<wire x1="-218.44" y1="139.7" x2="-215.9" y2="139.7" width="0.1524" layer="91"/>
-<pinref part="U$2" gate="G$1" pin="2"/>
-<wire x1="-215.9" y1="142.24" x2="-215.9" y2="139.7" width="0.1524" layer="91"/>
-<junction x="-215.9" y="139.7"/>
 </segment>
 <segment>
@@
 <wire x1="330.2" y1="127" x2="330.2" y2="124.46" width="0.1524" layer="91"/>
 </segment>
+<segment>
+<pinref part="U$1" gate="G$1" pin="P$1"/>
+<pinref part="GND12" gate="1" pin="GND"/>
+<wire x1="-218.44" y1="142.24" x2="-218.44" y2="139.7" width="0.1524" layer="91"/>
+</segment>
 </net>
 <net name="RESET" class="0">
@@
 </segment>
 <segment>
-<wire x1="-187.96" y1="160.02" x2="-215.9" y2="160.02" width="0.1524" layer="91"/>
-<pinref part="U$2" gate="G$1" pin="3"/>
-<wire x1="-215.9" y1="160.02" x2="-218.44" y2="160.02" width="0.1524" layer="91"/>
-<wire x1="-218.44" y1="152.4" x2="-218.44" y2="160.02" width="0.1524" layer="91"/>
-<junction x="-218.44" y="160.02"/>
-<pinref part="U$2" gate="G$1" pin="4"/>
-<wire x1="-215.9" y1="152.4" x2="-215.9" y2="160.02" width="0.1524" layer="91"/>
-<junction x="-215.9" y="160.02"/>
+<wire x1="-187.96" y1="160.02" x2="-218.44" y2="160.02" width="0.1524" layer="91"/>
 <pinref part="R3" gate="G$1" pin="1"/>
 <wire x1="-218.44" y1="160.02" x2="-218.44" y2="165.1" width="0.1524" layer="91"/>
 <label x="-210.82" y="160.02" size="1.778" layer="95"/>
 <pinref part="IC1" gate="G$1" pin="RESET"/>
+<pinref part="U$1" gate="G$1" pin="P$2"/>
+<wire x1="-218.44" y1="160.02" x2="-218.44" y2="157.48" width="0.1524" layer="91"/>
+<junction x="-218.44" y="160.02"/>
 </segment>
 </net>
@@
 <pinref part="SERIAL1" gate="J$1" pin="1"/>
 <wire x1="218.44" y1="50.8" x2="210.82" y2="50.8" width="0.1524" layer="91"/>
+<label x="210.82" y="50.8" size="1.778" layer="95"/>
 </segment>
 </net>
@@
 <pinref part="SERIAL1" gate="J$1" pin="2"/>
 <wire x1="218.44" y1="48.26" x2="210.82" y2="48.26" width="0.1524" layer="91"/>
+<label x="210.82" y="48.26" size="1.778" layer="95"/>
 </segment>
 </net>
@@
 <pinref part="SERIAL2" gate="J$1" pin="1"/>
 <wire x1="218.44" y1="35.56" x2="210.82" y2="35.56" width="0.1524" layer="91"/>
+<label x="210.82" y="35.56" size="1.778" layer="95"/>
 </segment>
 </net>
@@
 <pinref part="SERIAL2" gate="J$1" pin="2"/>
 <wire x1="218.44" y1="33.02" x2="210.82" y2="33.02" width="0.1524" layer="91"/>
+<label x="210.82" y="33.02" size="1.778" layer="95"/>
 </segment>
 </net>
@@
 <pinref part="PWM1" gate="G$1" pin="3"/>
 <wire x1="218.44" y1="109.22" x2="213.36" y2="109.22" width="0.1524" layer="91"/>
+<label x="210.82" y="109.22" size="1.778" layer="95"/>
 </segment>
 </net>
@@
 <pinref part="PWM1" gate="G$1" pin="4"/>
 <wire x1="218.44" y1="106.68" x2="213.36" y2="106.68" width="0.1524" layer="91"/>
+<label x="210.82" y="106.68" size="1.778" layer="95"/>
 </segment>
 </net>
@@
 <pinref part="PWM2" gate="G$1" pin="3"/>
 <wire x1="218.44" y1="88.9" x2="213.36" y2="88.9" width="0.1524" layer="91"/>
+<label x="210.82" y="88.9" size="1.778" layer="95"/>
 </segment>
 </net>
@@
 <pinref part="PWM2" gate="G$1" pin="4"/>
 <wire x1="218.44" y1="86.36" x2="213.36" y2="86.36" width="0.1524" layer="91"/>
+<label x="210.82" y="86.36" size="1.778" layer="95"/>
 </segment>
 </net>
@@
 <pinref part="PWM3" gate="G$1" pin="1"/>
 <wire x1="218.44" y1="71.12" x2="213.36" y2="71.12" width="0.1524" layer="91"/>
+<label x="210.82" y="71.12" size="1.778" layer="95"/>
 </segment>
 </net>
@@
 <pinref part="PWM3" gate="G$1" pin="2"/>
 <wire x1="218.44" y1="68.58" x2="213.36" y2="68.58" width="0.1524" layer="91"/>
+<label x="210.82" y="68.58" size="1.778" layer="95"/>
 </segment>
 </net>
@@
 <pinref part="PWM3" gate="G$1" pin="3"/>
 <wire x1="218.44" y1="66.04" x2="213.36" y2="66.04" width="0.1524" layer="91"/>
+<label x="210.82" y="66.04" size="1.778" layer="95"/>
 </segment>
 </net>
@@
 <pinref part="PWM3" gate="G$1" pin="4"/>
 <wire x1="218.44" y1="63.5" x2="213.36" y2="63.5" width="0.1524" layer="91"/>
+<label x="210.82" y="63.5" size="1.778" layer="95"/>
 </segment>
 </net>
@@
 <pinref part="PWM2" gate="G$1" pin="2"/>
 <wire x1="218.44" y1="91.44" x2="213.36" y2="91.44" width="0.1524" layer="91"/>
+<label x="210.82" y="91.44" size="1.778" layer="95"/>
 </segment>
 </net>
@@
 <pinref part="PWM2" gate="G$1" pin="1"/>
 <wire x1="218.44" y1="93.98" x2="213.36" y2="93.98" width="0.1524" layer="91"/>
+<label x="210.82" y="93.98" size="1.778" layer="95"/>
 </segment>
 </net>
@@
 </segment>
 </net>
+<net name="JTTDI" class="0">
+<segment>
+<pinref part="IC1" gate="G$1" pin="(ADC7/TDI)PF7"/>
+<pinref part="JTAG_CONNECTOR" gate="G$1" pin="C1"/>
+<wire x1="-116.84" y1="45.72" x2="-111.76" y2="45.72" width="0.1524" layer="91"/>
+<label x="-116.84" y="45.72" size="1.778" layer="95"/>
+</segment>
+</net>
+<net name="JTTDO" class="0">
+<segment>
+<pinref part="IC1" gate="G$1" pin="(ADC6/TDO)PF6"/>
+<pinref part="JTAG_CONNECTOR" gate="G$1" pin="C2"/>
+<wire x1="-116.84" y1="43.18" x2="-111.76" y2="43.18" width="0.1524" layer="91"/>
+<label x="-116.84" y="43.18" size="1.778" layer="95"/>
+</segment>
+</net>
+<net name="JTTMS" class="0">
+<segment>
+<pinref part="IC1" gate="G$1" pin="(ADC5/TMS)PF5"/>
+<pinref part="JTAG_CONNECTOR" gate="G$1" pin="C3"/>
+<wire x1="-116.84" y1="40.64" x2="-111.76" y2="40.64" width="0.1524" layer="91"/>
+<label x="-116.84" y="40.64" size="1.778" layer="95"/>
+</segment>
+</net>
+<net name="JTTCK" class="0">
+<segment>
+<pinref part="IC1" gate="G$1" pin="(ADC4/TCK)PF4"/>
+<pinref part="JTAG_CONNECTOR" gate="G$1" pin="C4"/>
+<wire x1="-116.84" y1="38.1" x2="-111.76" y2="38.1" width="0.1524" layer="91"/>
+<label x="-116.84" y="38.1" size="1.778" layer="95"/>
+</segment>
+</net>
