File: Arduino-Pro-v16.sch (EAGLE design)
At the start: 36 parts, among them IC1 ATMEGA1281-16AU, IC2 MCP170312MB, J1 FTDI Basic Programmer

Commit message: Started ordering the layout of the board
Parts:
- removed FRAME1: FRAME-LETTER, SparkFun-Aesthetics:FRAME-LETTER
Connections:
- removed net N$18: PWM3.1
- removed net N$19: PWM3.2
- removed net N$20: PWM3.3
- net PWM3A: now also PWM3.1
- net PWM3B: now also PWM3.2
- net PWM3C: now also PWM3.3
Changed lines of the file:
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@@
 <part name="GND7" library="SparkFun-Aesthetics" deviceset="GND" device=""/>
 <part name="GND9" library="SparkFun-Aesthetics" deviceset="GND" device=""/>
-<part name="FRAME1" library="SparkFun-Aesthetics" deviceset="FRAME-LETTER" device=""/>
 <part name="D1" library="DiscreteComponents" deviceset="DIODE-" device="DO-214AC"/>
 <part name="T1" library="DiscreteComponents" deviceset="FDN340P" device=""/>
@@
 <instance part="GND7" gate="1" x="213.36" y="43.18"/>
 <instance part="GND9" gate="1" x="210.82" y="27.94"/>
-<instance part="FRAME1" gate="G$1" x="-251.46" y="0"/>
-<instance part="FRAME1" gate="V" x="-104.14" y="0"/>
 <instance part="D1" gate="G$1" x="86.36" y="121.92" rot="R270"/>
 <instance part="T1" gate="A" x="71.12" y="116.84" rot="MR270"/>
@@
 </segment>
 </net>
-<net name="N$18" class="0">
+<net name="N$21" class="0">
+<segment>
+<pinref part="PWM3" gate="G$1" pin="4"/>
+<wire x1="218.44" y1="63.5" x2="213.36" y2="63.5" width="0.1524" layer="91"/>
+<label x="210.82" y="63.5" size="1.778" layer="95"/>
+</segment>
+</net>
+<net name="PWM0B" class="0">
+<segment>
+<pinref part="IC1" gate="G$1" pin="(OC0B)PG5"/>
+<wire x1="-116.84" y1="22.86" x2="-106.68" y2="22.86" width="0.1524" layer="91"/>
+<label x="-114.3" y="22.86" size="1.778" layer="95"/>
+</segment>
+<segment>
+<pinref part="PWM1" gate="G$1" pin="2"/>
+<wire x1="218.44" y1="111.76" x2="213.36" y2="111.76" width="0.1524" layer="91"/>
+<label x="210.82" y="111.76" size="1.778" layer="95"/>
+</segment>
+</net>
+<net name="PWM0A" class="0">
+<segment>
+<pinref part="IC1" gate="G$1" pin="(OC0A/OC1C/PCINT7)PB7"/>
+<wire x1="-116.84" y1="137.16" x2="-109.22" y2="137.16" width="0.1524" layer="91"/>
+<label x="-114.3" y="137.16" size="1.778" layer="95"/>
+</segment>
+<segment>
+<pinref part="PWM1" gate="G$1" pin="1"/>
+<wire x1="218.44" y1="114.3" x2="213.36" y2="114.3" width="0.1524" layer="91"/>
+<label x="210.82" y="114.3" size="1.778" layer="95"/>
+</segment>
+</net>
+<net name="PWM1B" class="0">
+<segment>
+<pinref part="IC1" gate="G$1" pin="(OC1B/PCINT6)PB6"/>
+<wire x1="-116.84" y1="134.62" x2="-109.22" y2="134.62" width="0.1524" layer="91"/>
+<label x="-114.3" y="134.62" size="1.778" layer="95"/>
+</segment>
+<segment>
+<pinref part="PWM2" gate="G$1" pin="2"/>
+<wire x1="218.44" y1="91.44" x2="213.36" y2="91.44" width="0.1524" layer="91"/>
+<label x="210.82" y="91.44" size="1.778" layer="95"/>
+</segment>
+</net>
+<net name="PWM1A" class="0">
+<segment>
+<pinref part="IC1" gate="G$1" pin="(OC1A/PCINT5)PB5"/>
+<wire x1="-116.84" y1="132.08" x2="-109.22" y2="132.08" width="0.1524" layer="91"/>
+<label x="-114.3" y="132.08" size="1.778" layer="95"/>
+</segment>
+<segment>
+<pinref part="PWM2" gate="G$1" pin="1"/>
+<wire x1="218.44" y1="93.98" x2="213.36" y2="93.98" width="0.1524" layer="91"/>
+<label x="210.82" y="93.98" size="1.778" layer="95"/>
+</segment>
+</net>
+<net name="PWM2A" class="0">
+<segment>
+<pinref part="IC1" gate="G$1" pin="(OC2A/PCINT4)PB4"/>
+<wire x1="-116.84" y1="129.54" x2="-109.22" y2="129.54" width="0.1524" layer="91"/>
+<label x="-114.3" y="129.54" size="1.778" layer="95"/>
+</segment>
+</net>
+<net name="PWM3C" class="0">
+<segment>
+<pinref part="IC1" gate="G$1" pin="(OC3C/INT5)PE5"/>
+<wire x1="-116.84" y1="63.5" x2="-106.68" y2="63.5" width="0.1524" layer="91"/>
+<label x="-114.3" y="63.5" size="1.778" layer="95"/>
+</segment>
+<segment>
+<pinref part="PWM3" gate="G$1" pin="3"/>
+<wire x1="218.44" y1="66.04" x2="213.36" y2="66.04" width="0.1524" layer="91"/>
+<label x="210.82" y="66.04" size="1.778" layer="95"/>
+</segment>
+</net>
+<net name="PWM3B" class="0">
+<segment>
+<pinref part="IC1" gate="G$1" pin="(OC3B/INT4)PE4"/>
+<wire x1="-116.84" y1="60.96" x2="-106.68" y2="60.96" width="0.1524" layer="91"/>
+<label x="-114.3" y="60.96" size="1.778" layer="95"/>
+</segment>
+<segment>
+<pinref part="PWM3" gate="G$1" pin="2"/>
+<wire x1="218.44" y1="68.58" x2="213.36" y2="68.58" width="0.1524" layer="91"/>
+<label x="210.82" y="68.58" size="1.778" layer="95"/>
+</segment>
+</net>
+<net name="PWM3A" class="0">
+<segment>
+<pinref part="IC1" gate="G$1" pin="(OC3A/AIN1)PE3"/>
+<wire x1="-116.84" y1="58.42" x2="-106.68" y2="58.42" width="0.1524" layer="91"/>
+<label x="-114.3" y="58.42" size="1.778" layer="95"/>
+</segment>
 <segment>
 <pinref part="PWM3" gate="G$1" pin="1"/>
@@
 </segment>
 </net>
-<net name="N$19" class="0">
-<segment>
-<pinref part="PWM3" gate="G$1" pin="2"/>
-<wire x1="218.44" y1="68.58" x2="213.36" y2="68.58" width="0.1524" layer="91"/>
-<label x="210.82" y="68.58" size="1.778" layer="95"/>
-</segment>
-</net>
-<net name="N$20" class="0">
-<segment>
-<pinref part="PWM3" gate="G$1" pin="3"/>
-<wire x1="218.44" y1="66.04" x2="213.36" y2="66.04" width="0.1524" layer="91"/>
-<label x="210.82" y="66.04" size="1.778" layer="95"/>
-</segment>
-</net>
-<net name="N$21" class="0">
-<segment>
-<pinref part="PWM3" gate="G$1" pin="4"/>
-<wire x1="218.44" y1="63.5" x2="213.36" y2="63.5" width="0.1524" layer="91"/>
-<label x="210.82" y="63.5" size="1.778" layer="95"/>
-</segment>
-</net>
-<net name="PWM0B" class="0">
-<segment>
-<pinref part="IC1" gate="G$1" pin="(OC0B)PG5"/>
-<wire x1="-116.84" y1="22.86" x2="-106.68" y2="22.86" width="0.1524" layer="91"/>
-<label x="-114.3" y="22.86" size="1.778" layer="95"/>
-</segment>
-<segment>
-<pinref part="PWM1" gate="G$1" pin="2"/>
-<wire x1="218.44" y1="111.76" x2="213.36" y2="111.76" width="0.1524" layer="91"/>
-<label x="210.82" y="111.76" size="1.778" layer="95"/>
-</segment>
-</net>
-<net name="PWM0A" class="0">
-<segment>
-<pinref part="IC1" gate="G$1" pin="(OC0A/OC1C/PCINT7)PB7"/>
-<wire x1="-116.84" y1="137.16" x2="-109.22" y2="137.16" width="0.1524" layer="91"/>
-<label x="-114.3" y="137.16" size="1.778" layer="95"/>
-</segment>
-<segment>
-<pinref part="PWM1" gate="G$1" pin="1"/>
-<wire x1="218.44" y1="114.3" x2="213.36" y2="114.3" width="0.1524" layer="91"/>
-<label x="210.82" y="114.3" size="1.778" layer="95"/>
-</segment>
-</net>
-<net name="PWM1B" class="0">
-<segment>
-<pinref part="IC1" gate="G$1" pin="(OC1B/PCINT6)PB6"/>
-<wire x1="-116.84" y1="134.62" x2="-109.22" y2="134.62" width="0.1524" layer="91"/>
-<label x="-114.3" y="134.62" size="1.778" layer="95"/>
-</segment>
-<segment>
-<pinref part="PWM2" gate="G$1" pin="2"/>
-<wire x1="218.44" y1="91.44" x2="213.36" y2="91.44" width="0.1524" layer="91"/>
-<label x="210.82" y="91.44" size="1.778" layer="95"/>
-</segment>
-</net>
-<net name="PWM1A" class="0">
-<segment>
-<pinref part="IC1" gate="G$1" pin="(OC1A/PCINT5)PB5"/>
-<wire x1="-116.84" y1="132.08" x2="-109.22" y2="132.08" width="0.1524" layer="91"/>
-<label x="-114.3" y="132.08" size="1.778" layer="95"/>
-</segment>
-<segment>
-<pinref part="PWM2" gate="G$1" pin="1"/>
-<wire x1="218.44" y1="93.98" x2="213.36" y2="93.98" width="0.1524" layer="91"/>
-<label x="210.82" y="93.98" size="1.778" layer="95"/>
-</segment>
-</net>
-<net name="PWM2A" class="0">
-<segment>
-<pinref part="IC1" gate="G$1" pin="(OC2A/PCINT4)PB4"/>
-<wire x1="-116.84" y1="129.54" x2="-109.22" y2="129.54" width="0.1524" layer="91"/>
-<label x="-114.3" y="129.54" size="1.778" layer="95"/>
-</segment>
-</net>
-<net name="PWM3C" class="0">
-<segment>
-<pinref part="IC1" gate="G$1" pin="(OC3C/INT5)PE5"/>
-<wire x1="-116.84" y1="63.5" x2="-106.68" y2="63.5" width="0.1524" layer="91"/>
-<label x="-114.3" y="63.5" size="1.778" layer="95"/>
-</segment>
-</net>
-<net name="PWM3B" class="0">
-<segment>
-<pinref part="IC1" gate="G$1" pin="(OC3B/INT4)PE4"/>
-<wire x1="-116.84" y1="60.96" x2="-106.68" y2="60.96" width="0.1524" layer="91"/>
-<label x="-114.3" y="60.96" size="1.778" layer="95"/>
-</segment>
-</net>
-<net name="PWM3A" class="0">
-<segment>
-<pinref part="IC1" gate="G$1" pin="(OC3A/AIN1)PE3"/>
-<wire x1="-116.84" y1="58.42" x2="-106.68" y2="58.42" width="0.1524" layer="91"/>
-<label x="-114.3" y="58.42" size="1.778" layer="95"/>
-</segment>
-</net>
