File: Co-Processor-v1.brd (EAGLE design)
At the start: 100 x 80 mm, 40 parts, among them IC1 ATMEGA1281-16AU, IC2 MCP170312MB, J1 FTDI Basic Programmer

Commit message: Routing
Parts:
- moved U$1 6.84 mm to (16.5, 62.2), turned to 0 degrees
- moved J1 5.24 mm to (8.89, 61.0)
- moved PWM1 5.24 mm to (8.89, 17.8)
- moved PWM2 5.24 mm to (8.89, 35.6)
- moved PWM3 5.24 mm to (8.89, 58.4)
- moved SPI_PIN 5.24 mm to (8.89, 38.1)
Routing:
- net 3V3: track 23.0 -> 56.5 mm, vias 0 -> 1
- net PWM0A: track 0.00 -> 27.2 mm
- net PWM0B: track 24.8 -> 45.1 mm, vias 1 -> 2
- net PWM1B: track 0.00 -> 15.4 mm
- net PWM1A: track 0.00 -> 14.6 mm
- net RESET: track 20.7 -> 28.9 mm
- net VCC: track 90.5 -> 97.4 mm, vias 1 -> 4
- net PWM3C: track 9.62 -> 15.2 mm
- net SCK: track 7.77 -> 13.4 mm
- net PWM3B: track 11.1 -> 16.0 mm
- net MOSI: track 7.92 -> 12.6 mm
- net MISO: track 8.64 -> 13.2 mm
- net PWM3A: track 12.6 -> 16.7 mm
- net TX0: track 16.2 -> 19.6 mm
- net RXI: track 17.7 -> 21.1 mm
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