File: Arduino-Pro-v17.brd (EAGLE design)
At the start: 39 x 53.3 mm, 39 parts, among them IC1 ATMEGA1281-16AU, IC2 MCP170312MB, J1 FTDI Basic Programmer

Commit message: Finished all routing, added pinouts for silkscreening on top of the board
Connections:
- removed net N$21: PWM3.4
- net GND: now also PWM3.4
- net PWM0A: now also PWM2.4; no longer PWM2.3
- net PWM0B: now also PWM2.3; no longer PWM2.4
Routing:
- net PWM0B: track 32.7 -> 30.2 mm
- net PWM0A: track 13.0 -> 15.2 mm, vias 2 -> 0
Other:
- board text added: "3V3"
- board text added: "5VIn"
- board text added: "ALTVin"
- board text added: "Co-Processor By Jason King ROV - X9 V1.0 11-2016"
- board text added: "DTR"
- board text added: "GND"
- board text added: "MISO"
- board text added: "MOSI"
- board text added: "PWM0A"
- board text added: "PWM0B"
- board text added: "PWM1A"
- board text added: "PWM1B"
- board text added: "PWM3A"
- board text added: "PWM3B"
- board text added: "PWM3C"
- board text added: "RXI"
- board text added: "SCK"
- board text added: "SCL"
- board text added: "SDA"
- board text added: "TCK"
- board text added: "TDI"
- board text added: "TDO"
- board text added: "TMS"
- board text added: "TX0"
- board text added: "VCC"
Changed lines of the file:
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@@
 <layer number="23" name="tOrigins" color="15" fill="1" visible="yes" active="yes"/>
 <layer number="24" name="bOrigins" color="15" fill="1" visible="yes" active="yes"/>
-<layer number="25" name="tNames" color="7" fill="1" visible="yes" active="yes"/>
-<layer number="26" name="bNames" color="7" fill="1" visible="yes" active="yes"/>
+<layer number="25" name="tNames" color="7" fill="1" visible="no" active="yes"/>
+<layer number="26" name="bNames" color="7" fill="1" visible="no" active="yes"/>
 <layer number="27" name="tValues" color="7" fill="1" visible="yes" active="yes"/>
 <layer number="28" name="bValues" color="7" fill="1" visible="yes" active="yes"/>
@@
 <vertex x="34.29" y="31.75"/>
 </polygon>
+<text x="9.2964" y="71.882" size="1.016" layer="21">GND</text>
+<text x="9.2964" y="69.342" size="1.016" layer="21">GND</text>
+<text x="9.2964" y="46.482" size="1.016" layer="21">GND</text>
+<text x="9.2964" y="49.022" size="1.016" layer="21">GND</text>
+<text x="39.0652" y="26.1874" size="1.016" layer="21">GND</text>
+<text x="9.6774" y="66.8528" size="1.016" layer="21">3V3</text>
+<text x="9.6774" y="61.6966" size="1.016" layer="21">TX0</text>
+<text x="9.779" y="64.2874" size="1.016" layer="21">RXI</text>
+<text x="9.4488" y="59.182" size="1.016" layer="21">DTR</text>
+<text x="9.1948" y="56.8706" size="0.6096" layer="21">PWM3A</text>
+<text x="9.2202" y="54.3052" size="0.6096" layer="21">PWM3B</text>
+<text x="9.1694" y="51.816" size="0.6096" layer="21">PWM3C</text>
+<text x="9.2202" y="34.036" size="0.6096" layer="21">PWM1A</text>
+<text x="9.1694" y="31.4452" size="0.6096" layer="21">PWM1B</text>
+<text x="9.1948" y="28.8798" size="0.6096" layer="21">PWM0B</text>
+<text x="9.271" y="26.4414" size="0.6096" layer="21">PWM0A</text>
+<text x="9.271" y="36.2712" size="1.016" layer="21">VCC</text>
+<text x="8.89" y="38.8874" size="1.016" layer="21">MISO</text>
+<text x="8.9408" y="41.3766" size="1.016" layer="21">MOSI</text>
+<text x="9.3218" y="43.9674" size="1.016" layer="21">SCK</text>
+<text x="38.8874" y="33.7312" size="1.016" layer="21">VCC</text>
+<text x="38.9636" y="31.3182" size="1.016" layer="21">SDA</text>
+<text x="39.0144" y="28.7274" size="1.016" layer="21">SCL</text>
+<text x="34.544" y="64.135" size="0.4064" layer="21" rot="R45">GND</text>
+<text x="34.6202" y="66.802" size="0.4064" layer="21" rot="R45">5VIn</text>
+<text x="34.036" y="61.4934" size="0.4064" layer="21" rot="R45">ALTVin</text>
+<text x="38.3032" y="36.4744" size="1.016" layer="21">Co-Processor
+By Jason King
+ROV - X9
+V1.0   11-2016</text>
+<text x="21.9202" y="67.7418" size="0.6096" layer="21">GND</text>
+<text x="24.5618" y="67.7164" size="0.6096" layer="21">TCK</text>
+<text x="27.051" y="67.7164" size="0.6096" layer="21">TMS</text>
+<text x="29.6672" y="67.7164" size="0.6096" layer="21">TDO</text>
+<text x="32.3342" y="67.691" size="0.6096" layer="21">TDI</text>
 </plain>
 <attributes>
@@
 <via x="16.51" y="45.72" extent="1-16" drill="0.6" diameter="0.508"/>
 <via x="34.29" y="49.53" extent="1-16" drill="0.6" diameter="0.508"/>
-<via x="43.18" y="31.75" extent="1-16" drill="0.6" diameter="0.508"/>
+<via x="43.18" y="29.21" extent="1-16" drill="0.6" diameter="0.508"/>
 <via x="26.67" y="62.23" extent="1-16" drill="0.6" diameter="0.508"/>
 <via x="44.45" y="73.66" extent="1-16" drill="0.6" diameter="0.508"/>
 <via x="39.37" y="71.12" extent="1-16" drill="0.6" diameter="0.508"/>
 <via x="16.51" y="73.66" extent="1-16" drill="0.6" diameter="0.508"/>
-<via x="21.59" y="29.21" extent="1-16" drill="0.6" diameter="0.508"/>
-<via x="43.18" y="33.02" extent="1-16" drill="0.6" diameter="0.508"/>
+<via x="20.32" y="27.94" extent="1-16" drill="0.6" diameter="0.508"/>
+<via x="43.18" y="35.56" extent="1-16" drill="0.6" diameter="0.508"/>
 <via x="34.29" y="41.91" extent="1-16" drill="0.6" diameter="0.508"/>
 <via x="27.94" y="41.91" extent="1-16" drill="0.6" diameter="0.508"/>
@@
 <contactref element="J2" pad="2"/>
 <contactref element="D2" pad="A"/>
+<contactref element="PWM3" pad="4"/>
 </signal>
 <signal name="RESET">
@@
 <wire x1="29.6164" y1="37.9476" x2="29.6037" y2="37.9603" width="0.4064" layer="1"/>
 </signal>
-<signal name="N$21">
-<contactref element="PWM3" pad="4"/>
-</signal>
 <signal name="PWM0B">
 <contactref element="IC1" pad="1"/>
-<contactref element="PWM2" pad="4"/>
 <wire x1="21.4503" y1="51.6255" x2="21.4503" y2="52.5145" width="0.4064" layer="1"/>
 <wire x1="21.4503" y1="52.5145" x2="21.5392" y2="52.6034" width="0.4064" layer="1"/>
@@
 <wire x1="24.13" y1="50.8" x2="24.13" y2="40.64" width="0.4064" layer="1"/>
 <wire x1="24.13" y1="40.64" x2="19.05" y2="35.56" width="0.4064" layer="1"/>
-<wire x1="19.05" y1="35.56" x2="19.05" y2="31.75" width="0.4064" layer="1"/>
-<wire x1="19.05" y1="31.75" x2="13.97" y2="26.67" width="0.4064" layer="1"/>
 <wire x1="22.3266" y1="52.6034" x2="24.13" y2="50.8" width="0.4064" layer="1"/>
+<contactref element="PWM2" pad="3"/>
+<wire x1="19.05" y1="35.56" x2="19.05" y2="34.29" width="0.4064" layer="1"/>
+<wire x1="19.05" y1="34.29" x2="13.97" y2="29.21" width="0.4064" layer="1"/>
 </signal>
 <signal name="PWM0A">
 <contactref element="IC1" pad="17"/>
-<contactref element="PWM2" pad="3"/>
-<wire x1="13.97" y1="29.21" x2="17.78" y2="33.02" width="0.4064" layer="1"/>
-<via x="17.78" y="33.02" extent="1-16" drill="0.6" diameter="0.508"/>
-<wire x1="17.78" y1="33.02" x2="20.32" y2="35.56" width="0.4064" layer="16"/>
-<via x="20.32" y="35.56" extent="1-16" drill="0.6" diameter="0.508"/>
-<wire x1="20.32" y1="35.56" x2="20.9042" y2="35.56" width="0.4064" layer="1"/>
-<wire x1="20.9042" y1="35.56" x2="23.3045" y2="37.9603" width="0.4064" layer="1"/>
+<contactref element="PWM2" pad="4"/>
+<wire x1="23.3045" y1="37.9603" x2="20.32" y2="34.9758" width="0.4064" layer="1"/>
+<wire x1="20.32" y1="34.9758" x2="20.32" y2="33.02" width="0.4064" layer="1"/>
+<wire x1="20.32" y1="33.02" x2="13.97" y2="26.67" width="0.4064" layer="1"/>
 </signal>
 <signal name="PWM1B">
@@
 </signal>
 <signal name="N$2">
-<via x="36.83" y="53.34" extent="1-16" drill="0.6" diameter="0.508"/>
+<via x="36.83" y="54.61" extent="1-16" drill="0.6" diameter="0.508"/>
 </signal>
 </signals>
@@
 </board>
 </drawing>
+<compatibility>
+<note version="6.3" minversion="6.2.2" severity="warning">
+Since Version 6.2.2 text objects can contain more than one line,
+which will not be processed correctly with this version.
+</note>
+</compatibility>
 </eagle>
