File: Arduino-Pro-v17.sch (EAGLE design)
At the start: 35 parts, among them IC1 ATMEGA1281-16AU, IC2 MCP170312MB, J1 FTDI Basic Programmer

Commit message: Added extra pinouts for JTAG, continued with layout
Parts:
- removed SERIAL1, SERIAL2: (no value), SparkFun-Connectors:M03PTH
- added C11, C12, C6, C7, C8, C9: 10uF, SparkFun-Passives:CAP0603-CAP
- added SV1: (no value), con-lsta:FE05-1
Connections:
- removed net N$2: SERIAL1.1
- removed net N$4: SERIAL1.2
- removed net N$6: SERIAL2.1
- removed net N$8: SERIAL2.2
- net GND: now also C11.2, C12.2, C6.2, C7.2, C8.2, C9.2, SV1.5; no longer SERIAL1.3, SERIAL2.3
- net JTTCK: now also SV1.4
- net JTTDI: now also SV1.1
- net JTTDO: now also SV1.2
- net JTTMS: now also SV1.3
- net MISO: now also IC1.(MISO/PCINT3)PB3
- net MOSI: now also IC1.(MOSI/PCINT2)PB2
- net SCK: now also IC1.(SCK/PCINT1)PB1
- net VCC: now also C11.1, C12.1, C6.1, C7.1, C8.1, C9.1
Other:
- moved on the sheet: C4, C5, JTAG_CONNECTOR, R3

Commit message: BC macz sukz
Parts:
- removed PWM1: (no value), SparkFun-Connectors:M04PTH
Connections:
- removed net N$12: PWM1.3
- removed net N$13: PWM1.4
- removed net N$17: PWM2.4
- removed net PWM1C: PWM2.3
- net PWM0A: now also PWM2.3; no longer PWM1.1
- net PWM0B: now also PWM2.4; no longer PWM1.2
Other:
- moved on the sheet: PWM2, PWM3
Changed lines of the file:
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@@
 <part name="PWM2" library="SparkFun-Connectors" deviceset="M04" device="PTH"/>
 <part name="PWM3" library="SparkFun-Connectors" deviceset="M04" device="PTH"/>
-<part name="PWM1" library="SparkFun-Connectors" deviceset="M04" device="PTH"/>
 <part name="D1" library="DiscreteComponents" deviceset="DIODE-" device="DO-214AC"/>
 <part name="T1" library="DiscreteComponents" deviceset="FDN340P" device=""/>
@@
 <instance part="P+1" gate="1" x="210.82" y="167.64"/>
 <instance part="P+5" gate="1" x="213.36" y="142.24"/>
-<instance part="PWM2" gate="G$1" x="223.52" y="91.44" rot="R180"/>
-<instance part="PWM3" gate="G$1" x="223.52" y="68.58" rot="R180"/>
-<instance part="PWM1" gate="G$1" x="223.52" y="111.76" rot="R180"/>
+<instance part="PWM2" gate="G$1" x="223.52" y="114.3" rot="R180"/>
+<instance part="PWM3" gate="G$1" x="223.52" y="91.44" rot="R180"/>
 <instance part="D1" gate="G$1" x="86.36" y="121.92" rot="R270"/>
 <instance part="T1" gate="A" x="71.12" y="116.84" rot="MR270"/>
@@
 </segment>
 </net>
-<net name="N$12" class="0">
-<segment>
-<pinref part="PWM1" gate="G$1" pin="3"/>
-<wire x1="218.44" y1="109.22" x2="213.36" y2="109.22" width="0.1524" layer="91"/>
-<label x="210.82" y="109.22" size="1.778" layer="95"/>
-</segment>
-</net>
-<net name="N$13" class="0">
-<segment>
-<pinref part="PWM1" gate="G$1" pin="4"/>
-<wire x1="218.44" y1="106.68" x2="213.36" y2="106.68" width="0.1524" layer="91"/>
-<label x="210.82" y="106.68" size="1.778" layer="95"/>
-</segment>
-</net>
-<net name="PWM1C" class="0">
-<segment>
-<pinref part="PWM2" gate="G$1" pin="3"/>
-<wire x1="218.44" y1="88.9" x2="213.36" y2="88.9" width="0.1524" layer="91"/>
-<label x="210.82" y="88.9" size="1.778" layer="95"/>
-</segment>
-</net>
-<net name="N$17" class="0">
-<segment>
-<pinref part="PWM2" gate="G$1" pin="4"/>
+<net name="N$21" class="0">
+<segment>
+<pinref part="PWM3" gate="G$1" pin="4"/>
 <wire x1="218.44" y1="86.36" x2="213.36" y2="86.36" width="0.1524" layer="91"/>
 <label x="210.82" y="86.36" size="1.778" layer="95"/>
-</segment>
-</net>
-<net name="N$21" class="0">
-<segment>
-<pinref part="PWM3" gate="G$1" pin="4"/>
-<wire x1="218.44" y1="63.5" x2="213.36" y2="63.5" width="0.1524" layer="91"/>
-<label x="210.82" y="63.5" size="1.778" layer="95"/>
 </segment>
 </net>
@@
 </segment>
 <segment>
-<pinref part="PWM1" gate="G$1" pin="2"/>
-<wire x1="218.44" y1="111.76" x2="213.36" y2="111.76" width="0.1524" layer="91"/>
-<label x="210.82" y="111.76" size="1.778" layer="95"/>
+<pinref part="PWM2" gate="G$1" pin="4"/>
+<wire x1="218.44" y1="109.22" x2="213.36" y2="109.22" width="0.1524" layer="91"/>
+<label x="210.82" y="109.22" size="1.778" layer="95"/>
 </segment>
 </net>
@@
 </segment>
 <segment>
-<pinref part="PWM1" gate="G$1" pin="1"/>
-<wire x1="218.44" y1="114.3" x2="213.36" y2="114.3" width="0.1524" layer="91"/>
-<label x="210.82" y="114.3" size="1.778" layer="95"/>
+<pinref part="PWM2" gate="G$1" pin="3"/>
+<wire x1="218.44" y1="111.76" x2="213.36" y2="111.76" width="0.1524" layer="91"/>
+<label x="210.82" y="111.76" size="1.778" layer="95"/>
 </segment>
 </net>
@@
 <segment>
 <pinref part="PWM2" gate="G$1" pin="2"/>
-<wire x1="218.44" y1="91.44" x2="213.36" y2="91.44" width="0.1524" layer="91"/>
-<label x="210.82" y="91.44" size="1.778" layer="95"/>
+<wire x1="218.44" y1="114.3" x2="213.36" y2="114.3" width="0.1524" layer="91"/>
+<label x="210.82" y="114.3" size="1.778" layer="95"/>
 </segment>
 </net>
@@
 <segment>
 <pinref part="PWM2" gate="G$1" pin="1"/>
-<wire x1="218.44" y1="93.98" x2="213.36" y2="93.98" width="0.1524" layer="91"/>
-<label x="210.82" y="93.98" size="1.778" layer="95"/>
+<wire x1="218.44" y1="116.84" x2="213.36" y2="116.84" width="0.1524" layer="91"/>
+<label x="210.82" y="116.84" size="1.778" layer="95"/>
 </segment>
 </net>
@@
 <segment>
 <pinref part="PWM3" gate="G$1" pin="3"/>
-<wire x1="218.44" y1="66.04" x2="213.36" y2="66.04" width="0.1524" layer="91"/>
-<label x="210.82" y="66.04" size="1.778" layer="95"/>
+<wire x1="218.44" y1="88.9" x2="213.36" y2="88.9" width="0.1524" layer="91"/>
+<label x="210.82" y="88.9" size="1.778" layer="95"/>
 </segment>
 </net>
@@
 <segment>
 <pinref part="PWM3" gate="G$1" pin="2"/>
-<wire x1="218.44" y1="68.58" x2="213.36" y2="68.58" width="0.1524" layer="91"/>
-<label x="210.82" y="68.58" size="1.778" layer="95"/>
+<wire x1="218.44" y1="91.44" x2="213.36" y2="91.44" width="0.1524" layer="91"/>
+<label x="210.82" y="91.44" size="1.778" layer="95"/>
 </segment>
 </net>
@@
 <segment>
 <pinref part="PWM3" gate="G$1" pin="1"/>
-<wire x1="218.44" y1="71.12" x2="213.36" y2="71.12" width="0.1524" layer="91"/>
-<label x="210.82" y="71.12" size="1.778" layer="95"/>
-</segment>
-</net>
+<wire x1="218.44" y1="93.98" x2="213.36" y2="93.98" width="0.1524" layer="91"/>
+<label x="210.82" y="93.98" size="1.778" layer="95"/>
+</segment>
+</net>

Commit message: Almost finished wiring
Parts:
- I2C_PIN: device SparkFun-Connectors:M05PTH -> SparkFun-Connectors:M04PTH
- J2: device SparkFun-Connectors:M01PTH -> SparkFun-Connectors:M02PTH
Connections:
- net 5VROV: now also J2.2
- net GND: no longer I2C_PIN.5
Changed lines of the file:
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@@
 <layer number="18" name="Vias" color="2" fill="1" visible="no" active="no"/>
 <layer number="19" name="Unrouted" color="6" fill="1" visible="no" active="no"/>
-<layer number="20" name="Dimension" color="6" fill="1" visible="no" active="no"/>
-<layer number="21" name="tPlace" color="16" fill="1" visible="no" active="no"/>
-<layer number="22" name="bPlace" color="14" fill="1" visible="no" active="no"/>
+<layer number="20" name="Dimension" color="15" fill="1" visible="no" active="no"/>
+<layer number="21" name="tPlace" color="7" fill="1" visible="no" active="no"/>
+<layer number="22" name="bPlace" color="7" fill="1" visible="no" active="no"/>
 <layer number="23" name="tOrigins" color="15" fill="1" visible="no" active="no"/>
 <layer number="24" name="bOrigins" color="15" fill="1" visible="no" active="no"/>
@@
 <layer number="49" name="Reference" color="7" fill="1" visible="no" active="no"/>
 <layer number="50" name="dxf" color="7" fill="1" visible="no" active="no"/>
-<layer number="51" name="tDocu" color="6" fill="1" visible="no" active="no"/>
+<layer number="51" name="tDocu" color="7" fill="1" visible="no" active="no"/>
 <layer number="52" name="bDocu" color="7" fill="1" visible="no" active="no"/>
 <layer number="53" name="tGND_GNDA" color="7" fill="9" visible="no" active="no"/>
@@
 <part name="C2" library="SparkFun-Capacitors" deviceset="CAP" device="0603-CAP"/>
 <part name="GND2" library="SparkFun" deviceset="GND" device=""/>
-<part name="I2C_PIN" library="SparkFun-Connectors" deviceset="M05" device="PTH"/>
+<part name="I2C_PIN" library="SparkFun-Connectors" deviceset="M04" device="PTH"/>
 <part name="SPI_PIN" library="SparkFun-Connectors" deviceset="M05" device="PTH"/>
 <part name="GND3" library="SparkFun-Aesthetics" deviceset="GND" device=""/>
@@
 <part name="C4" library="SparkFun-Capacitors" deviceset="CAP" device="0603-CAP"/>
 <part name="IC2" library="linear" deviceset="MCP1703*" device="MB" technology="12"/>
-<part name="J2" library="SparkFun-Connectors" deviceset="M01" device="PTH"/>
+<part name="J2" library="SparkFun-Connectors" deviceset="M02" device="PTH"/>
 <part name="C6" library="SparkFun-Passives" deviceset="CAP" device="0603-CAP" value="10uF"/>
 <part name="C7" library="SparkFun-Passives" deviceset="CAP" device="0603-CAP" value="10uF"/>
@@
 <instance part="C2" gate="G$1" x="-198.12" y="157.48" rot="R270"/>
 <instance part="GND2" gate="1" x="-208.28" y="152.4"/>
-<instance part="I2C_PIN" gate="G$1" x="226.06" y="160.02" rot="R180"/>
+<instance part="I2C_PIN" gate="G$1" x="223.52" y="162.56" rot="R180"/>
 <instance part="SPI_PIN" gate="G$1" x="226.06" y="134.62" rot="R180"/>
 <instance part="GND3" gate="1" x="210.82" y="152.4"/>
@@
 <pinref part="I2C_PIN" gate="G$1" pin="4"/>
 <wire x1="218.44" y1="157.48" x2="210.82" y2="157.48" width="0.1524" layer="91"/>
-<pinref part="I2C_PIN" gate="G$1" pin="5"/>
-<wire x1="218.44" y1="154.94" x2="210.82" y2="154.94" width="0.1524" layer="91"/>
 <wire x1="210.82" y1="157.48" x2="210.82" y2="154.94" width="0.1524" layer="91"/>
 <pinref part="GND3" gate="1" pin="GND"/>
-<junction x="210.82" y="154.94"/>
 </segment>
 <segment>
@@
 <label x="81.28" y="152.4" size="1.778" layer="95"/>
 </segment>
-</net>
+<segment>
+<pinref part="J2" gate="G$1" pin="2"/>
+<wire x1="50.8" y1="119.38" x2="55.88" y2="119.38" width="0.1524" layer="91"/>
+<label x="53.34" y="119.38" size="1.778" layer="95"/>
+</segment>
+</net>
